File: 909_noise.kicad_sch (KiCad schematic)
At the start: 23 parts, among them J1 1x4 Header, J2 1x3 Header, J3 ${MPN}, SW1 ${MPN}, U1 ${MPN}, U2 ${MPN}, U4 NE5532

Commit message: r0.3 schematic/layout
- change active filter values to filter at lower freq
- add raw 3V3 output
- add two types of level shifters to 12V
- add passively filtered 12V output
Parts:
- removed J2: 1x3 Header, Connector_PinHeader_2.54mm:PinHeader_1x03_P2.54mm_Vertical, symbol gkeeth-dblib:Connectors/CONN0003
- removed R2, R3: ${Resistance}, Resistor_SMD:R_0603_1608Metric, symbol gkeeth-dblib:Resistors/R0341
- added C10, C11, C8: ${Capacitance}, Capacitor_SMD:C_0603_1608Metric, symbol gkeeth-dblib:Capacitors/C0085
- added C9: ${Capacitance}, Capacitor_SMD:C_0603_1608Metric, symbol gkeeth-dblib:Capacitors/C0041
- added J2: 1x10 Header, Connector_PinHeader_2.54mm:PinHeader_1x10_P2.54mm_Vertical, symbol gkeeth-dblib:Connectors/CONN0010
- added R2, R3, R7: ${Resistance}, Resistor_SMD:R_0603_1608Metric, symbol gkeeth-dblib:Resistors/R0386
- added U3: ${MPN}, Package_SO:SOIC-16W_5.3x10.2mm_P1.27mm, symbol gkeeth-dblib:Logic/LOGIC0003
- added U5: ${MPN}, Package_SO:SOIC-16_3.9x9.9mm_P1.27mm, symbol gkeeth-dblib:Logic/LOGIC0002
Connections:
- net +12V: now also C11.2, C8.2, U3.16 (V_{DD}), U5.1 (VCC), U5.13 (Select), U5.16 (VDD)
- net +3.3V: now also C10.2, U3.1 (V_{CC}), U3.2 (ENABLE_A)
- net GND: now also C10.1, C11.1, C8.1, C9.2, J2.10 (Pin_10), J2.2 (Pin_2), J2.4 (Pin_4), J2.6 (Pin_6), J2.8 (Pin_8), U3.10 (C), U3.14 (D), U3.15 (ENABLE_D), U3.6 (B), U3.7 (ENABLE_B), U3.8 (V_{SS}), U3.9 (ENABLE_C), U5.11 (Ein), U5.14 (Fin), U5.5 (Bin), U5.7 (Cin), U5.8 (VSS), U5.9 (Din)
- net noise_3v3: now also J2.7 (Pin_7), R2.2, U3.3 (A), U5.3 (Ain)
- net at C7.1, U4.3 (+), U4.5 (+): now also R3.1
- net at C6.1: now also R2.1, R3.2
- net noise_12v renamed noise_12v_active_filt
- net noise_12v_active_filt: now also J2.1 (Pin_1)
- new net noise_12v_40109: J2.9 (Pin_9), U3.4 (E)
- new net noise_12v_4504: J2.3 (Pin_3), R7.2, U5.2 (Aout)
- new net noise_12v_4504_filt: C9.1, J2.5 (Pin_5), R7.1
- no-connect marks 3 -> 12
Other:
- moved on the sheet: C1, C2, C3, C5, D1, J3, R1, SW1, U1, U2
